File: kicad-v5/1ump-master/1ump-master.sch (KiCad schematic (older format))
At the start: 3 parts

Commit message: Add MCU to master board.
Parts:
- added C? (x4): 100n, symbol C
- added C? (x4): 22p, symbol C
- added U?: STM32F103C8Tx, Housings_QFP:LQFP-48_7x7mm_Pitch0.5mm, symbol STM32F103C8Tx
- added Y?: 8MHz, symbol Crystal
- added Y?: 32kHz, symbol Crystal_GND23
Connections:
- net labels added: +3.3V, +5V, FT-DTR, FT-RX, FT-TX, GND, MIS, MOS, TWCL-RX, TWCL-SB, TWCL-TX
- wire segments 0 -> 21

Commit message: Add STM32f103C8T6 and FT232RQ.
Parts:
- added C?: 10n, symbol C
- added C? (x2): 100n, symbol C
- added C?: 4.7u, symbol CP
- added C?: 10u, symbol C
- added C?: 10u, symbol CP
- added D?: LED-WHITE, symbol LED_ALT
- added D?: LED-GREEN, symbol LED_ALT
- added D? (x2): LED-YELLOW, symbol LED_ALT
- added J?: Conn_01x04, symbol Conn_01x04
- added J?: USB_B, symbol USB_B
- added JP? (x2): Jumper_NC_Dual, symbol Jumper_NC_Dual
- added L?: Bead, symbol Ferrite_Bead
- added R? (x4): 1k, symbol R
- added R? (x2): 100k, symbol R
- added R? (x2): 10k, symbol R
- added R? (x2): 27R, symbol R
- added U?: FT232RQ, symbol FT232RQ
Connections:
- net labels added: +5VA, BLINK, BOOT0, BOOT1, D+, D-, SWCLK, SWDIO
- wire segments 21 -> 40
- no-connect marks 0 -> 20
Other:
- moved on the sheet: C?, J?, U?, Y?

Commit message: Add master circuit.
Parts:
- removed J?: USB_B, symbol USB_B
- added C1, C2: 10u, symbol CP_Small
- added C16, C4: 10u, symbol C_Small
- added C24: 100n, symbol C-RESCUE-1ump-master
- added C3, C6, C7, C8: 22p, symbol C_Small
- added C5: 330u, symbol CP_Small
- added D1, D2, D3, D4: 1N4007, symbol D_Small_ALT
- added D5, D6: LED_YELLOW, symbol LED_Small_ALT
- added J1: Conn_01x03, symbol Conn_01x03
- added J2: DC_JACK, symbol DC_JACK
- added J7, J8: USB_B, symbol USB_B
- added Q1: IRFR5305, symbol Q_PMOS_GDSD
- added R1, R2, R3, R4, R5, R6, R7, R8: 1k, symbol R_Small
- added R10, R9: 1k, symbol R-RESCUE-1ump-master
- added R21, R22: 27R, symbol R-RESCUE-1ump-master
- added U1: AMS1117-3.3, symbol AMS1117-3.3
- added U2, U6: OR_GATE, symbol OR_GATE
- added U3: NAND_GATE, symbol NAND_GATE
- added U4, U5: Buffer_Noninverting_1G, symbol Buffer_Noninverting_1G
- C11, C12, C13, C14, C15, C17, C18, C19, C20, C22, C23, C9: renamed from C?; symbol C -> C-RESCUE-1ump-master
- R11, R12, R13, R14, R15, R16, R17, R18, R19, R20: renamed from R?; symbol R -> R-RESCUE-1ump-master
- gave numbers to parts that had none: 17
Connections:
- net labels added: +5VP, MASPROGSEL, MASTFRX, MASTFTX
- wire segments 40 -> 106
- no-connect marks 20 -> 40
Other:
- moved on the sheet: C10, C11, C12, C13, C14, C15, C17, C18, C19, C20, C21, C22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

Commit message: Add changes to slave board.
Parts:
- added C?: 10n, symbol C-RESCUE-1ump-master
- added D?: LED-GREEN, symbol LED_ALT
- added J? (x6): Conn_01x03, symbol Connector:Conn_01x03
- added J? (x3): Conn_01x05, symbol Connector:Conn_01x05
- added L?: Bead, symbol Ferrite_Bead
- added R?: 1k, symbol R-RESCUE-1ump-master
Connections:
- net labels added: +5VD
- wire segments 106 -> 107
- no-connect marks 40 -> 39
Other:
- moved on the sheet: J3, J4
