File: kicad-v5/1ump-slave/1ump-slave.sch (KiCad schematic (older format))
At the start: 34 parts

Commit message: In progress...
Parts:
- removed J?: Conn_01x04, symbol Connector:Conn_01x04
- added C?: 100n, symbol Device:C
- added J?: Conn_02x03_Odd_Even, symbol Connector:Conn_02x03_Odd_Even
- added J?: Conn_01x06, symbol Connector:Conn_01x06
- added U?: ATtiny44A-MU, Package_DFN_QFN:QFN-20-1EP_4x4mm_P0.5mm_EP2.25x2.25mm, symbol MCU_Microchip_ATtiny:ATtiny44A-MU
Connections:
- net labels added: +3.3V, +5V, MIS, MISO, MOS, MOSI, RST, SCL
- wire segments 82 -> 89
- no-connect marks 0 -> 2
Other:
- moved on the sheet: Q?

Commit message: Added MCU ATtiny44A, LCD driver not done.
Parts:
- removed D? (x2): 1N4007, Diode_SMD:D_SOD-123, symbol Device:D_ALT
- removed Q?: 2N7002, Package_TO_SOT_SMD:SOT-23, symbol Transistor_FET:2N7002
- removed R? (x2): 1k, Resistor_SMD:R_0805_2012Metric, symbol Device:R
- removed U? (x2): SN74LVC1G125DCKR, Package_TO_SOT_SMD:SOT-353_SC-70-5, symbol Custom_Logic_74xxx:Buffer_Noninverting_1G
- added C1, C10, C11, C13, C6, C7, C9: 10n, symbol Device:C
- added C3, C4: 15p, symbol Device:C
- added C5, C8: 100n, symbol Device:C
- added J6: Conn_01x03, symbol Connector:Conn_01x03
- added JP1: Jumper, symbol Device:Jumper
- added Q1, Q2, Q7, Q8: 2N7002, Package_TO_SOT_SMD:SOT-23, symbol Transistor_FET:2N7002
- added R1: 1M, Resistor_SMD:R_0805_2012Metric, symbol Device:R
- added R10, R11, R13, R14, R16, R18, R2, R3, R4, R6, R8, R9: 10k, Resistor_SMD:R_0805_2012Metric, symbol Device:R
- added R5: 0, Resistor_SMD:R_0805_2012Metric, symbol Device:R
- added RN1: R_Pack07-1k, symbol Device:R_Pack07
- added U14: ELD-426SYGWA, Display_7Segment:ELD_426XXXX, symbol Display_Character:ELD-426SYGWA
- added U15: SN74LVC1G00DCKR, Package_TO_SOT_SMD:SOT-353_SC-70-5, symbol Custom_Logic_74xxx:NAND_GATE
- added U2, U5: 74HC74, symbol 74xx:74HC74
- added U4: 74AUC1G74, symbol 74xGxx:74AUC1G74
- added U7: 4511, symbol 4xxx_IEEE:4511
- added Y1: 16MHz - SMD-3225_4P, symbol Device:Crystal_GND24
- R12: renamed from R?; value 1k -> 10k
- gave numbers to parts that had none: 29
Connections:
- net labels added: DIS-COUNT, DREF, INC-IN, JMOSI, NDREF, XTAL1, XTAL2
- net labels removed: ALERT, CHECK, TECL-RX
- wire segments 89 -> 170
- no-connect marks 2 -> 1
Other:
- moved on the sheet: J3, J4, Q3, Q4, Q5, Q6, U1

Commit message: Slave board complit.
Parts:
- removed D2: 1N4007, Diode_SMD:D_SOD-123, symbol Device:D_ALT
- removed J3: Conn_01x06, symbol Connector:Conn_01x06
- removed U15: SN74LVC1G00DCKR, Package_TO_SOT_SMD:SOT-353_SC-70-5, symbol Custom_Logic_74xxx:NAND_GATE
- removed U4: 74AUC1G74, symbol 74xGxx:74AUC1G74
- added C13, C?: 100n, symbol Device:C
- added J3: Conn_01x05, symbol Connector:Conn_01x05
- added R10, R11, R16: 10k, Resistor_SMD:R_0805_2012Metric, symbol Device:R
- added R24: 10k, symbol Device:R
- added SW1: SW_Push, symbol Switch:SW_Push
- added unit 1 of U4
- added unit 1 of U8
- R15: value 1k -> 10k
- renumbered C13 to C14, R10 to R12, R11 to R13, R12 to R14, R13 to R17, R14 to R18, R16 to R20, R17 to R21, R18 to R22, R19 to R23, U16 to U15, U17 to U16, U5 to U4, U6 to U5, U7 to U6, U8 to U7, U5 to U8
Connections:
- net labels added: SEG1, SEG2, SEL-SEG, SET-SEG
- net labels removed: DREF, JMOSI, NDREF
- no-connect marks 1 -> 3
Other:
- moved on the sheet: Q1, Q2, Q4, Q6, Q7, Q8, U2A, U2B, U8B

Commit message: Add MCU to master board.
Parts:
- gave numbers to parts that had none: 1
- renumbered C9 to C10, C10 to C11, C11 to C12, C12 to C13, C13 to C14, C14 to C15, C6 to C7, C7 to C8, C8 to C9, D3 to D2, R20 to R19, R21 to R20, R22 to R21, R23 to R22, R24 to R23
Connections:
- wire segments 170 -> 142

Commit message: Add changes to slave board.
Parts:
- removed C6, C9: 100n, symbol Device:C
- removed C8: 10n, symbol Device:C
- removed J1, J2: Conn_01x03, symbol Connector:Conn_01x03
- removed J3: Conn_01x05, symbol Connector:Conn_01x05
- removed J4: Conn_02x03_Odd_Even, symbol Connector:Conn_02x03_Odd_Even
- removed R10, R11, R12, R13, R15, R8: 10k, Resistor_SMD:R_0805_2012Metric, symbol Device:R
- removed RN1: R_Pack07-1k, symbol Device:R_Pack07
- removed U2, U4, U8: 74HC74, symbol 74xx:74HC74
- removed U6: 4511, symbol 4xxx_IEEE:4511
- added C11, C12: 10u, Capacitors_SMD:C_0805, symbol CP_Small
- added C14, C2, C3, C4, C7: 100n, Capacitors_SMD:C_0805, symbol Device:C
- added J1: Conn_02x03_Odd_Even, Pin_Headers:Pin_Header_Straight_2x03_Pitch2.54mm, symbol Conn_02x03_Odd_Even
- added J2: Conn_02x02_Odd_Even, Pin_Headers:Pin_Header_Straight_2x02_Pitch2.54mm, symbol Conn_02x02_Odd_Even
- added J3: Conn_01x02, Pin_Headers:Pin_Header_Angled_1x02_Pitch2.54mm, symbol Conn_01x02
- added J6: Conn_01x06, Connectors_JST:JST_PH_S6B-PH-K_06x2.00mm_Angled, symbol Conn_01x06
- added JP2: Jumper, Resistors_SMD:R_0805, symbol Device:Jumper
- added R1, R2, R6, R7: 10k, Resistors_SMD:R_0805, symbol Device:R
- added RN1: R_Pack08-330R, Resistors_SMD:R_Cat16-8, symbol R_Pack08
- added U1, U2, U3, U4: 74HC175, Housings_SOIC:SOIC-16_3.9x9.9mm_Pitch1.27mm, symbol 74HC175
- added U10: 74HC74_SOIC14, Housings_SOIC:SOIC-14_3.9x8.7mm_Pitch1.27mm, symbol 74HC74_SOIC14
- added U7: 74HC244, Housings_SOIC:SOIC-20W_7.5x12.8mm_Pitch1.27mm, symbol 74HC244
- added U9: AMS1117-3.3, TO_SOT_Packages_SMD:SOT-223, symbol AMS1117-3.3
- C1: value 10n -> 100n; footprint (none) -> Capacitors_SMD:C_0805
- C10: renamed from C3; footprint (none) -> Capacitors_SMD:C_0805
- C13: renamed from C4; footprint (none) -> Capacitors_SMD:C_0805
- C15: renamed from C11; footprint (none) -> Capacitors_SMD:C_0805
- C16: renamed from C15; footprint (none) -> Capacitors_SMD:C_0805
- C17: renamed from C10; footprint (none) -> Capacitors_SMD:C_0805
- C18: renamed from C12; footprint (none) -> Capacitors_SMD:C_0805
- C19: renamed from C13; footprint (none) -> Capacitors_SMD:C_0805
- C5: renamed from C2; footprint (none) -> Capacitors_SMD:C_0805
- C6: renamed from C5; footprint (none) -> Capacitors_SMD:C_0805
- C8: renamed from C7; footprint (none) -> Capacitors_SMD:C_0805
- C9: renamed from C14; footprint (none) -> Capacitors_SMD:C_0805
- D1: footprint (none) -> LEDs:LED_0805
- D2: footprint Diode_SMD:D_SOD-123 -> Diodes_SMD:D_0805
- J4: renamed from J5; footprint (none) -> Pin_Headers:Pin_Header_Angled_1x07_Pitch2.54mm
- J5: renamed from J6; footprint (none) -> Pin_Headers:Pin_Header_Angled_1x03_Pitch2.54mm
- JP1: footprint (none) -> Resistors_SMD:R_0805
- Q1, Q2: footprint Package_TO_SOT_SMD:SOT-23 -> TO_SOT_Packages_SMD:SOT-23
- Q3: renamed from Q7; footprint Package_TO_SOT_SMD:SOT-23 -> TO_SOT_Packages_SMD:SOT-23
- Q4: renamed from Q8; footprint Package_TO_SOT_SMD:SOT-23 -> TO_SOT_Packages_SMD:SOT-23
- Q5: renamed from Q3; footprint Package_TO_SOT_SMD:SOT-23 -> TO_SOT_Packages_SMD:SOT-23
- Q6: renamed from Q5; footprint Package_TO_SOT_SMD:SOT-23 -> TO_SOT_Packages_SMD:SOT-23
- Q7: renamed from Q4; footprint Package_TO_SOT_SMD:SOT-23 -> TO_SOT_Packages_SMD:SOT-23
- Q8: renamed from Q6; footprint Package_TO_SOT_SMD:SOT-23 -> TO_SOT_Packages_SMD:SOT-23
- R10: renamed from R7; footprint Resistor_SMD:R_0805_2012Metric -> Resistors_SMD:R_0805
- R11: renamed from R19; footprint Resistor_SMD:R_0805_2012Metric -> Resistors_SMD:R_0805
- R12: renamed from R21; footprint Resistor_SMD:R_0805_2012Metric -> Resistors_SMD:R_0805
- R13: renamed from R23; footprint (none) -> Resistors_SMD:R_0805
- R14: renamed from R1; footprint Resistor_SMD:R_0805_2012Metric -> Resistors_SMD:R_0805
- R15: renamed from R5; footprint Resistor_SMD:R_0805_2012Metric -> Resistors_SMD:R_0805
- R16, R17, R18, R20, R3, R4, R9: footprint Resistor_SMD:R_0805_2012Metric -> Resistors_SMD:R_0805
- R19: renamed from R14; footprint Resistor_SMD:R_0805_2012Metric -> Resistors_SMD:R_0805
- R21: renamed from R22; footprint (none) -> Resistors_SMD:R_0805
- R5: renamed from R2; footprint Resistor_SMD:R_0805_2012Metric -> Resistors_SMD:R_0805
- R8: renamed from R6; footprint Resistor_SMD:R_0805_2012Metric -> Resistors_SMD:R_0805
- SW1: footprint (none) -> Buttons_Switches_THT:SW_Tactile_SPST_Angled_PTS645Vx39-2LFS
- U11: renamed from U5; footprint Package_TO_SOT_SMD:SOT-353_SC-70-5 -> TO_SOT_Packages_SMD:SOT-353_SC-70-5
- U12: renamed from U15; footprint Package_TO_SOT_SMD:SOT-353_SC-70-5 -> TO_SOT_Packages_SMD:SOT-353_SC-70-5
- U13: renamed from U11; footprint Package_TO_SOT_SMD:SOT-353_SC-70-5 -> TO_SOT_Packages_SMD:SOT-353_SC-70-5
- U14: renamed from U7; footprint Package_TO_SOT_SMD:SOT-353_SC-70-5 -> TO_SOT_Packages_SMD:SOT-353_SC-70-5
- U15: renamed from U9; footprint Package_TO_SOT_SMD:SOT-353_SC-70-5 -> TO_SOT_Packages_SMD:SOT-353_SC-70-5
- U16: renamed from U10; footprint Package_TO_SOT_SMD:SOT-353_SC-70-5 -> TO_SOT_Packages_SMD:SOT-353_SC-70-5
- U17: renamed from U12; footprint Package_TO_SOT_SMD:SOT-353_SC-70-5 -> TO_SOT_Packages_SMD:SOT-353_SC-70-5
- U18: renamed from U13; footprint Package_TO_SOT_SMD:SOT-353_SC-70-5 -> TO_SOT_Packages_SMD:SOT-353_SC-70-5
- U19: renamed from U16; footprint Package_TO_SOT_SMD:SOT-353_SC-70-5 -> TO_SOT_Packages_SMD:SOT-353_SC-70-5
- U5: renamed from U1; footprint Package_DFN_QFN:QFN-20-1EP_4x4mm_P0.5mm_EP2.25x2.25mm -> Housings_DFN_QFN:QFN-20-1EP_4x4mm_Pitch0.5mm
- U6: renamed from U3; footprint Package_TO_SOT_SMD:SOT-353_SC-70-5 -> TO_SOT_Packages_SMD:SOT-353_SC-70-5
- Y1: footprint (none) -> Crystals:Crystal_SMD_0603-4pin_6.0x3.5mm
- renumbered U14 to U8
Connections:
- net labels added: SHIFT-IN, SHIFT-SHOW, SHIFT-VALUE, SOS, USER-INPUT
- net labels removed: DIS-COUNT, ECHO, INC-IN, SEL-SEG, SET-SEG, VCC
- wire segments 142 -> 250
- no-connect marks 3 -> 18
Other:
- note added: "COMMUNICATION BUS"
- note added: "MASTER-SLAVE BUS"
- note added: "MCU CONNECTOR"
- note added: "SPI CONNETOR"
- note added: "VOLTAGE SELECT"
- moved on the sheet: Q1, Q2, Q3, Q4, Q5, Q6, Q7, Q8, U5
