File: kicad-v5/1ump_master_rev1-x/1ump_master_rev1-x.sch (KiCad schematic (older format))
At the start: 105 parts, among them U1 74HC74, U2 74HC74, U3 74HC74, U4 74HC74, U5 74HC74, U6 74HC74, U7 74HC74, U8 74HC74

Commit message: Add TWCL testing.
Parts:
- removed C? (x2): 100n, symbol Device:C
- removed D? (x2): LED_YELLOW, symbol Device:LED_ALT
- removed J?: USB_B, symbol Connector:USB_B
- removed L?: Ferrite_Bead, symbol Device:Ferrite_Bead
- removed R?: 10k, symbol Device:R
- removed R? (x2): 330, symbol Device:R
- removed R? (x2): 27, symbol Device:R
- removed U?: CP2102, symbol cp2102:CP2102
- removed U?: 74HC00, symbol 74xx:74HC00
- added D?: LED_GREEN, symbol Device:LED_ALT
- added J?: USB_B, symbol Connector:USB_B
- added L?: Ferrite_Bead, symbol Device:Ferrite_Bead
- added R? (x2): 27, symbol Device:R
- added R?: 1k, symbol Device:R
Connections:
- net labels added: STM_D+, STM_D-
- net labels removed: LOG_RX, LOG_TX
- wire segments 342 -> 327
- no-connect marks 37 -> 29
